File: Dev-kit-multiboards.kicad_sch (KiCad schematic)
At the start: 25 parts, among them J1 Conn_01x04_Socket, J2 Conn_01x04_Socket, J3 Conn_01x02_Socket, J4 Conn_01x19_Socket, J5 Conn_01x19_Socket, J6 Conn_01x02_Socket, J7 Conn_01x02_Socket, J8 Conn_02x17_Counter_Clockwise, SW1 SW_Push, SW2 SW_Push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

Commit message: component placement
Parts:
- added RGB2: WS2812B, WS2812B:WS2812B, symbol WS2812B:WS2812B
- BUTTON1: renamed from SW1; footprint (none) -> Button_Switch_SMD:SW_Push_1P1T_NO_6x6mm_H9.5mm
- BUTTON2: renamed from SW2; footprint (none) -> Button_Switch_SMD:SW_Push_1P1T_NO_6x6mm_H9.5mm
- BUTTON3: renamed from SW3; footprint (none) -> Button_Switch_SMD:SW_Push_1P1T_NO_6x6mm_H9.5mm
- BUZZER1: renamed from BZ1; footprint (none) -> Buzzer_Beeper:Buzzer_12x9.5RM7.6
- C1: renamed from C2; footprint (none) -> Capacitor_SMD:C_1206_3216Metric
- C2: renamed from C3; footprint (none) -> Capacitor_SMD:C_1206_3216Metric
- C3: renamed from C1; footprint (none) -> Capacitor_SMD:C_1206_3216Metric
- J1, J2: footprint (none) -> Connector_PinHeader_2.54mm:PinHeader_1x04_P2.54mm_Vertical
- J3, J6, J7: footprint (none) -> Connector_PinHeader_2.54mm:PinHeader_1x02_P2.54mm_Vertical
- J4, J5: footprint (none) -> Connector_PinSocket_2.54mm:PinSocket_1x19_P2.54mm_Vertical
- J8: footprint (none) -> Connector_PinHeader_2.54mm:PinHeader_2x17_P2.54mm_Vertical
- LED1: renamed from D1; footprint (none) -> LED_SMD:LED_1206_3216Metric
- LED2: renamed from D2; footprint (none) -> LED_SMD:LED_1206_3216Metric
- R1: renamed from R2; value 100k -> 10k; footprint (none) -> Resistor_SMD:R_1206_3216Metric
- R2: renamed from R3; value 100k -> 10k; footprint (none) -> Resistor_SMD:R_1206_3216Metric
- R3: renamed from R1; value 100k -> 10k; footprint (none) -> Resistor_SMD:R_1206_3216Metric
- R4, R5: value 1K -> 300; footprint (none) -> Resistor_SMD:R_1206_3216Metric
- R6, R7: footprint (none) -> Resistor_SMD:R_1206_3216Metric
- RGB1: renamed from LED1; footprint (none) -> WS2812B:WS2812B
Connections:
- net +3.3V: now also LED1.2 (A), RGB2.1-VDD (VDD)
- net Earth: now also RGB2.3-GND (GND)
- net IO12: now also RGB2.4-DIN (DI)
- net IO32: no longer LED1.2 (A)
- no-connect marks 1 -> 2
Other:
- note added: "10k: C3018037 1206 300: C104757 1206 100nF: C377067 1206"
- note added: "1TS005F-2500-5001 C255812"
- note added: "C2935901"
- note added: "C541858"
- note added: "RGB WS2812B"
- note added: "TMB12A03 C96222"
- note added: "XL-3216SURC C965822"
- note added: "XL-5050RGBC-WS2812B C2843785"
- note removed: "RGB"
- moved on the sheet: BUZZER1, LED1, LED2, R4, R5, RGB1

Commit message: Component placement ESP32
Parts:
- removed J8: Conn_02x17_Counter_Clockwise, Connector_PinHeader_2.54mm:PinHeader_2x17_P2.54mm_Vertical, symbol Connector_Generic:Conn_02x16_Counter_Clockwise
- added J12: Conn_01x02_Socket, Connector_PinHeader_2.54mm:PinHeader_1x02_P2.54mm_Vertical, symbol Connector:Conn_01x02_Socket
- added J8, J9: Conn_01x19, Connector_PinHeader_2.54mm:PinHeader_1x19_P2.54mm_Vertical, symbol Connector_Generic:Conn_01x19
Connections:
- net +3.3V: now also J8.1 (Pin_1)
- net +5V: now also J8.19 (Pin_19)
- net BUTTON1: now also J9.16 (Pin_16)
- net BUTTON2: now also J9.17 (Pin_17)
- net BUTTON3: now also J9.18 (Pin_18)
- net Buzzer: now also J9.15 (Pin_15)
- net CLK: now also J9.9 (Pin_9)
- net CS: now also J9.10 (Pin_10)
- net DAC_1: now also J8.9 (Pin_9)
- net DAC_2: now also J8.10 (Pin_10)
- net EN_ESP32: now also J8.2 (Pin_2)
- net Earth: now also J8.14 (Pin_14), J9.1 (Pin_1), J9.7 (Pin_7)
- net IO0: now also J9.14 (Pin_14)
- net IO1: now also J9.4 (Pin_4)
- net IO10: now also J12.1 (Pin_1), J8.17 (Pin_17)
- net IO11: now also J12.2 (Pin_2), J8.18 (Pin_18)
- net IO12: now also J8.13 (Pin_13)
- net IO13: now also J8.15 (Pin_15)
- net IO14: now also J8.12 (Pin_12)
- net IO16: now also J9.12 (Pin_12)
- net IO17: now also J9.11 (Pin_11)
- net IO19: now also J9.8 (Pin_8)
- net IO21: now also J9.6 (Pin_6)
- net IO22: now also J9.3 (Pin_3)
- net IO23: now also J9.2 (Pin_2)
- net IO27: now also J8.11 (Pin_11)
- net IO3: now also J9.5 (Pin_5)
- net IO32: now also J8.7 (Pin_7)
- net IO33: now also J8.8 (Pin_8)
- net IO34: now also J8.5 (Pin_5)
- net IO35: now also J8.6 (Pin_6)
- net IO39: now also J8.4 (Pin_4)
- net IO6: now also J9.19 (Pin_19)
- net IO9: now also J8.16 (Pin_16)
- net ADC1_0 renamed ADC1
- net ADC1: now also J8.3 (Pin_3)
- net ADC2_0 renamed ADC2
- net ADC2: now also J9.13 (Pin_13)
Other:
- note added: "PWM"
- moved on the sheet: BUZZER1, J1, J2, J3, J4, J5, J6, J7, LED1, LED2, R4, R5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

Commit message: Final version
Parts:
- removed R6, R7: 10K, Resistor_SMD:R_1206_3216Metric, symbol Device:R
- added J10: USB_B_Micro, Connector_USB:USB_Micro-B_Molex-105017-0001, symbol Connector:USB_B_Micro
- added JP1: Jumper_2_Bridged, Connector_PinHeader_2.54mm:PinHeader_1x02_P2.54mm_Vertical, symbol Jumper:Jumper_2_Bridged
- BUTTON1, BUTTON2, BUTTON3: LCSC Part Number (none) -> C255812
- BUZZER1: LCSC Part Number (none) -> C96222
- C1, C2, C3: LCSC Part Number (none) -> C377067
- J1, J2: LCSC Part Number (none) -> C6332197
- J12, J3, J6, J7: LCSC Part Number (none) -> C2685144
- J4, J5: LCSC Part Number (none) -> C2894942
- J8, J9: LCSC Part Number (none) -> C2897382
- LED1, LED2: LCSC Part Number (none) -> C965822
- R1, R2, R3: LCSC Part Number (none) -> C3018037
- R4, R5: LCSC Part Number (none) -> C104757
- RGB1, RGB2: LCSC Part Number (none) -> C2843785
Connections:
- net +5V: now also J10.1 (VBUS)
- net Buzzer: now also JP1.1 (A); no longer BUZZER1.1 (-)
- net Earth: now also J10.5 (GND), J10.6 (Shield)
- new net: BUZZER1.1 (-), JP1.2 (B)
- no-connect marks 2 -> 5
Other:
- moved on the sheet: BUZZER1
